File: CM5IO_top/CM5IO_top.kicad_pcb (KiCad board)
At the start: 2 copper layers, 50.3 x 56.3 mm, 58 parts, among them J1 USB_C_Receptacle_USB2.0, J10 J_DShot600_FC, J3 J_PSU_EN, J4 J_ESP_DBG_UART, J7 J_FC_UART, J8 THD-20-R, J9 J_DShot600_ESC, Q1 AO3401A, Q2 Q_NPN_BEC, Q3 Q_NPN_BEC, Q4 AO3401A, SW1 SW_RESET, SW2 SW_BOOT, SW3 FORCE_PWR, U1 ESP32-S3-WROOM-1, U2 Wio-SX1262, U3 AP7361C-33E, U4 AP7361C-33E

Commit message: Upload final gerbers with personal touch TM
Parts:
- removed H2: MountingHole, MountingHole:MountingHole_2.7mm_M2.5_DIN965
Routing:
- net GND: track 44.0 -> 47.3 mm, vias 60 -> 94
